File: SuperNinePin.kicad_pcb (KiCad board)
At the start: 2 copper layers, 63.3 x 53 mm, 25 parts, among them J3 Atari, Q1 2N3904, U2 74HC4040, U3 NE555P, U5 74HC595, U6 74HC595, U7 ULN2803A, U8 74HC74, U9 4051

Commit message: Adds gerbers, crude enclosure
Parts:
- removed C3, C8, C9: 1 uF, Capacitor_THT:C_Disc_D3.0mm_W1.6mm_P2.50mm
- removed U5, U6: 74HC595, Package_DIP:DIP-16_W7.62mm
- removed U7: ULN2803A, Package_DIP:DIP-18_W7.62mm
- removed U8: 74HC74, Package_DIP:DIP-14_W7.62mm
- added D1: FIRE, LED_THT:LED_D3.0mm, F.Cu at (206.1, 65.3)
- added J2: SNES, SuperNintendo:SNESController, F.Cu at (143.4, 52.9)
- added Q2: BS170, Package_TO_SOT_THT:TO-92_Inline_Wide, F.Cu at (183.6, 39.9)
- added Q3: BS170, Package_TO_SOT_THT:TO-92_Inline_Wide, F.Cu at (146.7, 37.6)
- added R10: 100R, Resistor_THT:R_Axial_DIN0207_L6.3mm_D2.5mm_P10.16mm_Horizontal, F.Cu at (198.6, 57.8)
- added R11: 100R, Resistor_THT:R_Axial_DIN0207_L6.3mm_D2.5mm_P10.16mm_Horizontal, F.Cu at (198.6, 54.5)
- added R12: 100R, Resistor_THT:R_Axial_DIN0207_L6.3mm_D2.5mm_P10.16mm_Horizontal, F.Cu at (198.6, 51.2)
- added R13: 100R, Resistor_THT:R_Axial_DIN0207_L6.3mm_D2.5mm_P10.16mm_Horizontal, F.Cu at (198.6, 47.9)
- added R14: 100R, Resistor_THT:R_Axial_DIN0207_L6.3mm_D2.5mm_P10.16mm_Horizontal, F.Cu at (198.6, 44.6)
- added R15: 470R, Resistor_THT:R_Axial_DIN0207_L6.3mm_D2.5mm_P10.16mm_Horizontal, F.Cu at (201.3, 66.3)
- added R7: 100K, Resistor_THT:R_Axial_DIN0207_L6.3mm_D2.5mm_P10.16mm_Horizontal, F.Cu at (164.7, 40.3)
- added R8: 10K, Resistor_THT:R_Axial_DIN0207_L6.3mm_D2.5mm_P10.16mm_Horizontal, F.Cu at (146.8, 43.8)
- added R9: 100R, Resistor_THT:R_Axial_DIN0207_L6.3mm_D2.5mm_P10.16mm_Horizontal, F.Cu at (198.6, 61.1)
- added REF**: OSHW-Logo2_7.3x6mm_SilkScreen, Symbol:OSHW-Logo2_7.3x6mm_SilkScreen, F.Cu at (201.9, 70.7)
- added U1: CD4060BE, Package_DIP:DIP-16_W7.62mm, F.Cu at (150.2, 50.9)
- C1: value 4.7 nF -> 68 pF; footprint Capacitor_THT:C_Disc_D3.0mm_W1.6mm_P2.50mm -> Capacitor_THT:C_Disc_D3.4mm_W2.1mm_P2.50mm
- C2: value 100 nF -> 10 µF; footprint Capacitor_THT:C_Disc_D3.0mm_W1.6mm_P2.50mm -> Capacitor_THT:C_Radial_D5.0mm_H5.0mm_P2.00mm
- J3: footprint Connector_Dsub:DSUB-9_Socket_EdgeMount_P2.77mm -> Connector_Dsub:DSUB-9_Pins_Horizontal_P2.77x2.84mm_EdgePinOffset4.94mm_Housed_MountingHolesOffset4.94mm
- Q1: value 2N3904 -> BS170
- R1: value 680R -> 10K
- R2: value 2.7K -> 10K
- R4: value 1K -> 470R
- R5: value 330R -> 1K
- R6: value 330R -> 470R
- U2: value 74HC4040 -> TPIC6595; footprint Package_DIP:DIP-16_W7.62mm -> Package_DIP:DIP-20_W7.62mm
- U3: value NE555P -> TPIC6595; footprint Package_DIP:DIP-8_W7.62mm -> Package_DIP:DIP-20_W7.62mm
- U9: value 4051 -> CD4051
- moved D2 98.3 mm to (208.7, 40.6), turned to 180 degrees
- moved R6 60.1 mm to (191.1, 40.3)
- moved R5 56.4 mm to (164.7, 36.8), turned to 180 degrees
- moved R4 52.7 mm to (180.6, 37.0), turned to 180 degrees
- moved U2 51.2 mm to (172.1, 63.2), turned to 90 degrees
- moved R3 45.5 mm to (180.6, 40.3), turned to 180 degrees
- moved C4 45.1 mm to (149.1, 40.9)
- moved U3 44.6 mm to (172.0, 50.9), turned to 90 degrees
- moved C6 43.6 mm to (174.8, 53.3)
- moved Q1 43.0 mm to (163.2, 67.5)
- moved C1 40.2 mm to (167.5, 38.1), turned to -90 degrees
- moved C7 36.3 mm to (175.7, 65.7), turned to 180 degrees
- moved C5 35.7 mm to (150.1, 53.3)
- moved C2 30.7 mm to (183.1, 68.3), turned to 90 degrees
- moved R2 27.1 mm to (150.5, 69.6)
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Connections:
- C1 pad 1: Net-(U3-THR) -> Net-(C1-Pad1)
- C1 pad 2: GND -> Net-(U1-C_{SET})
- C2 pad 1: Net-(U3-CV) -> +5V
- J3 pad 6: /TRIGGER -> /BUTTON1
- Q1 pad 1: GND -> /Turbo_Trigger
- Q1 pad 2: Net-(Q1-B) -> Net-(Q1-G)
- Q1 pad 3: Net-(Q1-C) -> GND
- R1 pad 1: Net-(U3-THR) -> +5V
- R1 pad 2: Net-(U3-DIS) -> /SNES_A
- R2 pad 1: Net-(U3-DIS) -> +5V
- R2 pad 2: +5V -> /SNES_X
- R3 pad 1: Net-(Q1-C) -> Net-(Q2-D)
- R4 pad 1: Net-(Q1-B) -> Net-(Q2-G)
- R5 pad 1: /TURBO -> Net-(C1-Pad1)
- U2 pad 1: unconnected-(U2-Q11-Pad1) -> GND
- U2 pad 10: /SNES_Clock -> GND
- U2 pad 12: unconnected-(U2-Q8-Pad12) -> /SNES_Latch
- U2 pad 13: unconnected-(U2-Q7-Pad13) -> /SNES_Clock
- U2 pad 14: /Turbo_Fire_CLK -> /SNES_R
- U2 pad 15: unconnected-(U2-Q10-Pad15) -> /SNES_L
- U2 pad 16: +5V -> /SNES_X
- U2 pad 2: unconnected-(U2-Q5-Pad2) -> +5V
- U2 pad 3: /SNES_Latch -> Net-(Q2-D)
- U2 pad 8: GND -> +5V
- U2 pad 9: unconnected-(U2-Q0-Pad9) -> GND
- U3 pad 2: Net-(U3-THR) -> +5V
- U3 pad 3: /SNES_Clock -> Net-(U2-SER_OUT)
- U3 pad 4: +5V -> /SNES_Right
- U3 pad 5: Net-(U3-CV) -> /SNES_Left
- U3 pad 6: Net-(U3-THR) -> /SNES_Down
- U3 pad 7: Net-(U3-DIS) -> /SNES_Up
- U9 pad 10: /~{TURBO} -> /SNES_X
- U9 pad 12: /Turbo_Fire_CLK -> GND
- U9 pad 13: GND -> /Turbo_Fire
- U9 pad 14: GND -> /Turbo_Fire
- U9 pad 15: GND -> +5V
- U9 pad 3: /Turbo_Trigger -> Net-(Q1-G)
- U9 pad 5: +5V -> GND
- U9 pad 9: /TURBO -> GND
Routing:
- net +5V: track 0.00 -> 246.4 mm
- net /SNES_Clock: track 0.00 -> 82.8 mm
- net /SNES_Latch: track 0.00 -> 72.7 mm
- net /SNES_Up: track 0.00 -> 56.9 mm
- net /Turbo_Trigger: track 0.00 -> 48.2 mm
- net /SNES_Data: track 0.00 -> 44.9 mm
- net /SNES_X: track 0.00 -> 41.2 mm
- net /SNES_A: track 0.00 -> 29.8 mm
- net Net-(Q2-D): track 0.00 -> 27.8 mm
- net /SNES_B: track 0.00 -> 21.3 mm
- net /SNES_Right: track 0.00 -> 20.3 mm
- net Net-(Q3-G): track 0.00 -> 19.9 mm
- net /SNES_Left: track 0.00 -> 18.6 mm
- net /SNES_Down: track 0.00 -> 18.2 mm
- net Net-(Q1-G): track 0.00 -> 17.4 mm
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- added copper zone on B.Cu, net GND
- added copper zone on F.Cu, net GND
Other:
- board size 63.3 x 53 mm -> 91.6 x 42.6 mm
- board text added: "+"
- board text added: "SuperNinePin"
